File: hardware/mainboard/mr-mainboard.kicad_sch (KiCad schematic)
At the start: 0 parts

Commit message: Core power, disp and camera wiring
Signed-off-by: David Shah <dave@ds0.me>
Other:
- added sheet Cam_Disp (mipi.kicad_sch)
- added sheet FPGA Power (fpga_pwr.kicad_sch)
