File: hardware/frontboard/meowality_front.kicad_sch (KiCad schematic)
At the start: 39 parts

Commit message: Add PCIe and camera to front board
Signed-off-by: gatecat <gatecat@ds0.me>
Parts:
- added C?: 1µ, symbol Device:C_Small
- added C?: 1n, symbol Device:C_Small
- added C? (x2): 12p, symbol Device:C_Small
- added C?: 4.7µ, symbol Device:C_Small
- added CAM?: PI_CAM_22P, symbol meowality:PI_CAM_22P
- added FB?: Ferrite_Bead_Small, symbol Device:Ferrite_Bead_Small
- added P?: M2_SOCKET_E, symbol meowality:M2_SOCKET_E
- added R? (x4): 2k2, symbol Device:R_Small
- added R?: 10k, symbol Device:R_Small
- added R? (x2): 0R, symbol Device:R_Small
- added R?: 200k, symbol Device:R_Small
- added U?: PCA9306, symbol Interface:PCA9306
- added U?: Si52112-B, symbol meowality:Si52112-B
- added Y?: 25MHz, symbol Device:Crystal_GND24_Small
Connections:
- net +1V8PL: now also R?.1, R?.1, U?.2 (VREF1)
- net +3V3PS: now also CAM?.22 (CAM_3V3), FB?.1, P?.2 (3.3V), P?.4 (3.3V), P?.72 (3.3V), P?.74 (3.3V), R?.1, R?.1, R?.1
- net CSI0_CLK+: now also CAM?.9 (CAM_CK+)
- net CSI0_CLK-: now also CAM?.8 (CAM_CK-)
- net CSI0_D0+: now also CAM?.3 (CAM_D0+)
- net CSI0_D0-: now also CAM?.2 (CAM_D0-)
- net CSI0_D1+: now also CAM?.6 (CAM_D1+)
- net CSI0_D1-: now also CAM?.5 (CAM_D1-)
- net CSI0_D2+: now also CAM?.12 (CAM_D2+)
- net CSI0_D2-: now also CAM?.11 (CAM_D2-)
- net CSI0_D3+: now also CAM?.15 (CAM_D3+)
- net CSI0_D3-: now also CAM?.14 (CAM_D3-)
- net FRONT_SCL: now also R?.2, U?.4 (SDA1)
- net FRONT_SDA: now also R?.2, U?.3 (SCL1)
- net GND: now also J?.B65, C?.2, C?.2, C?.2, C?.2, C?.2, CAM?.1 (GND), CAM?.10 (GND), CAM?.13 (GND), CAM?.16 (GND), CAM?.19 (GND), CAM?.4 (GND), CAM?.7 (GND), CAM?.M, P?.1 (GND), P?.18 (GND), P?.33 (GND), P?.39 (GND), P?.45 (GND), P?.51 (GND), P?.57 (GND), P?.63 (GND), P?.69 (GND), P?.7 (GND), P?.75 (GND), P?.M, R?.2, U?.11 (Vss), U?.4 (Vss), U?.5 (Vss), Y?.2, Y?.4
- net PCIE_C2M_L0+: now also P?.35 (PER0+)
- net PCIE_C2M_L0-: now also P?.37 (PER0-)
- net PCIE_C2M_L1+: now also P?.59 (PER1+)
- net PCIE_C2M_L1-: now also P?.61 (PER1-)
- net PCIE_M2C_L0+: now also P?.41 (PET0+)
- net PCIE_M2C_L0-: now also P?.43 (PET0-)
- net PCIE_M2C_L1+: now also P?.65 (PET1+)
- net PCIE_M2C_L1-: now also P?.67 (PET1-)
- net PCIE_REFCLK+: now also U?.8 (DIFF2+)
- net PCIE_REFCLK-: now also U?.9 (DIFF2-)
- net PCIE_~{PERST}: now reaches J?.B66
- net PCIE_~{PERST}: now also P?.52 (~{PERST0})
- net CAM_PWR_EN: now reaches J?.B67
- net CAM_PWR_EN: now also CAM?.17 (CAM_IO0), R?.1
- net FRONT_CAM_~{RST}: no longer names the net of J?.A27
- new net: CAM?.21 (CAM_SDA), R?.2, U?.5 (SDA2)
- new net: CAM?.20 (CAM_SCL), R?.2, U?.6 (SCL2)
- new net: C?.1, R?.2, U?.7 (VREF2), U?.8 (EN)
- new net: C?.1, C?.1, FB?.2, U?.1 (Vdd), U?.10 (Vdd)
- new net: C?.1, U?.3 (XIN), Y?.1
- new net: C?.1, U?.2 (XOUT), Y?.3
- new net REFCLK+: P?.47 (REFCLK0+), R?.2
- new net REFCLK-: P?.49 (REFCLK0-), R?.2
- new net REFCLKO1+: R?.1, U?.6 (DIFF1+)
- new net REFCLKO1-: R?.1, U?.7 (DIFF1-)
- no-connect marks 1 -> 42

Commit message: Add IMU
Signed-off-by: gatecat <gatecat@ds0.me>
Parts:
- added C? (x2): 1µ, symbol Device:C_Small
- added C?: 10µ, symbol Device:C_Small
- added U?: MMC5883MA, Package_LGA:LGA-16_3x3mm_P0.5mm, symbol Sensor_Magnetic:MMC5883MA
Connections:
- net +1V8PL: now also C?.1, U?.13 (VDDIO)
- net +3V3PS: now also C?.2, U?.2 (VDD)
- net FRONT_SCL: now also R?.2, U?.3 (SCL1), U?.1 (SCL); no longer R?.2, U?.4 (SDA1)
- net FRONT_SDA: now also R?.2, U?.4 (SDA1), U?.16 (SDA); no longer R?.2, U?.3 (SCL1)
- net GND: now also U?.1 (GND), C?.1, C?.2, C?.2, U?.11 (GND), U?.9 (GND)
- new net: C?.1, U?.10 (CAP)
- no-connect marks 42 -> 43

Commit message: Fixing various front and top board issues
Signed-off-by: gatecat <gatecat@ds0.me>
Parts:
- added C1: 1µ, symbol Device:C_Small
- added J2: LED, symbol Connector_Generic:Conn_01x04
- added U1: 74LVC2T45DC, Package_SO:VSSOP-8_2.3x2mm_P0.5mm, symbol Logic_LevelTranslator:74LVC2T45DC
- gave numbers to parts that had none: 62
Connections:
- net +1V8PL: now also U1.1 (VCCA), U1.5 (DIR)
- net +3V3PS: now also J1.A69, J1.B68, J1.B69
- net +5V: now also C1.1, J2.1 (Pin_1), U1.8 (VCCB)
- net DSI1A_D0+: no longer J1.A7, LCD1.11 (DSI_D0-_A)
- net FRONT_LED0: now also U1.2 (1A)
- net FRONT_LED1: now also U1.3 (2A)
- net GND: now also C1.2, J2.4 (Pin_4), U1.4 (GND); no longer J1.A69, J1.B68, J1.B69
- new net DSI1A_D0-: J1.A7, LCD1.11 (DSI_D0-_A)
- new net LED0: J2.2 (Pin_2), U1.7 (1B)
- new net LED1: J2.3 (Pin_3), U1.6 (2B)
- no-connect marks 43 -> 47
